File: driver.kicad_sch (KiCad schematic)
At the start: 5 parts, among them U2 74AHCT125

Commit message: all one layer added usb
Parts:
- renumbered R2 to R4, R3 to R5, R4 to R6, R5 to R7, U2 to U4
Changed lines of the file:
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@@
 		(dnp no)
 		(fields_autoplaced yes)
-		(property "Reference" "U2"
+		(property "Reference" "U4"
 			(at 120.65 77.47 0)
 			(effects
@@
 			(project ""
 				(path "/4f28ee59-d9ac-4dfb-922f-af5c6097cb64/b37b9310-7296-4533-8f70-fa9a758099d6"
-					(reference "U2")
+					(reference "U4")
 					(unit 3)
 				)
@@
 		(dnp no)
 		(fields_autoplaced yes)
-		(property "Reference" "R5"
+		(property "Reference" "R7"
 			(at 132.08 104.14 90)
 			(effects
@@
 			(project "wpiwaNDWSID"
 				(path "/4f28ee59-d9ac-4dfb-922f-af5c6097cb64/b37b9310-7296-4533-8f70-fa9a758099d6"
-					(reference "R5")
+					(reference "R7")
 					(unit 1)
 				)
@@
 		(dnp no)
 		(fields_autoplaced yes)
-		(property "Reference" "U2"
+		(property "Reference" "U4"
 			(at 120.65 101.6 0)
 			(effects
@@
 			(project ""
 				(path "/4f28ee59-d9ac-4dfb-922f-af5c6097cb64/b37b9310-7296-4533-8f70-fa9a758099d6"
-					(reference "U2")
+					(reference "U4")
 					(unit 4)
 				)
@@
 		(dnp no)
 		(fields_autoplaced yes)
-		(property "Reference" "R2"
+		(property "Reference" "R4"
 			(at 132.08 33.02 90)
 			(effects
@@
 			(project ""
 				(path "/4f28ee59-d9ac-4dfb-922f-af5c6097cb64/b37b9310-7296-4533-8f70-fa9a758099d6"
-					(reference "R2")
+					(reference "R4")
 					(unit 1)
 				)
@@
 		(dnp no)
 		(fields_autoplaced yes)
-		(property "Reference" "U2"
+		(property "Reference" "U4"
 			(at 88.9 71.1199 0)
 			(effects
@@
 			(project ""
 				(path "/4f28ee59-d9ac-4dfb-922f-af5c6097cb64/b37b9310-7296-4533-8f70-fa9a758099d6"
-					(reference "U2")
+					(reference "U4")
 					(unit 5)
 				)
@@
 		(dnp no)
 		(fields_autoplaced yes)
-		(property "Reference" "U2"
+		(property "Reference" "U4"
 			(at 120.65 30.48 0)
 			(effects
@@
 			(project ""
 				(path "/4f28ee59-d9ac-4dfb-922f-af5c6097cb64/b37b9310-7296-4533-8f70-fa9a758099d6"
-					(reference "U2")
+					(reference "U4")
 					(unit 1)
 				)
@@
 		(dnp no)
 		(fields_autoplaced yes)
-		(property "Reference" "R4"
+		(property "Reference" "R6"
 			(at 132.08 80.01 90)
 			(effects
@@
 			(project "wpiwaNDWSID"
 				(path "/4f28ee59-d9ac-4dfb-922f-af5c6097cb64/b37b9310-7296-4533-8f70-fa9a758099d6"
-					(reference "R4")
+					(reference "R6")
 					(unit 1)
 				)
@@
 		(dnp no)
 		(fields_autoplaced yes)
-		(property "Reference" "R3"
+		(property "Reference" "R5"
 			(at 132.08 57.15 90)
 			(effects
@@
 			(project "wpiwaNDWSID"
 				(path "/4f28ee59-d9ac-4dfb-922f-af5c6097cb64/b37b9310-7296-4533-8f70-fa9a758099d6"
-					(reference "R3")
+					(reference "R5")
 					(unit 1)
 				)
@@
 		(dnp no)
 		(fields_autoplaced yes)
-		(property "Reference" "U2"
+		(property "Reference" "U4"
 			(at 120.65 54.61 0)
 			(effects
@@
 			(project ""
 				(path "/4f28ee59-d9ac-4dfb-922f-af5c6097cb64/b37b9310-7296-4533-8f70-fa9a758099d6"
-					(reference "U2")
+					(reference "U4")
 					(unit 2)
 				)

Commit message: rev 2
Connections:
- net LED1_IN: now also U4.5; no longer U4.2
- net LED2_IN: now also U4.2; no longer U4.5
- net LED3_IN: now also U4.12; no longer U4.9
- net LED4_IN: now also U4.9; no longer U4.12
- net at U4.8: now also R7.1; no longer R6.1
- net at U4.11: now also R6.1; no longer R7.1
- net at R4.1: now also U4.6; no longer U4.3
- net at R5.1: now also U4.3; no longer U4.6
Other:
- moved on the sheet: R4, R5, R6, R7
Changed lines of the file:
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@@
 	(generator_version "9.0")
 	(paper "A4")
+	(junction
+		(at 128.27 110.49)
+		(diameter 0)
+		(color 0 0 0 0)
+	)
+	(wire
+		(pts
+			(xy 130.81 86.36) (xy 128.27 86.36)
+		)
+		(stroke
+			(width 0)
+			(type default)
+		)
+	)
+	(wire
+		(pts
+			(xy 110.49 110.49) (xy 113.03 110.49)
+		)
+		(stroke
+			(width 0)
+			(type default)
+		)
+	)
+	(wire
+		(pts
+			(xy 127 110.49) (xy 128.27 110.49)
+		)
+		(stroke
+			(width 0)
+			(type default)
+		)
+	)
+	(wire
+		(pts
+			(xy 128.27 110.49) (xy 134.62 110.49)
+		)
+		(stroke
+			(width 0)
+			(type default)
+		)
+	)
 	(hierarchical_label "V5.0"
 		(shape bidirectional)
@@
 	(hierarchical_label "LED3_IN"
 		(shape bidirectional)
+		(at 110.49 110.49 180)
+		(effects
+			(font
+				(size 1.27 1.27)
+			)
+			(justify right)
+		)
+	)
+	(hierarchical_label "LED2_IN"
+		(shape bidirectional)
+		(at 113.03 39.37 180)
+		(effects
+			(font
+				(size 1.27 1.27)
+			)
+			(justify right)
+		)
+	)
+	(hierarchical_label "LED2_OUT"
+		(shape bidirectional)
+		(at 135.89 39.37 0)
+		(effects
+			(font
+				(size 1.27 1.27)
+			)
+			(justify left)
+		)
+	)
+	(hierarchical_label "GND"
+		(shape bidirectional)
+		(at 120.65 45.72 270)
+		(effects
+			(font
+				(size 1.27 1.27)
+			)
+			(justify right)
+		)
+	)
+	(hierarchical_label "LED4_IN"
+		(shape bidirectional)
 		(at 113.03 86.36 180)
 		(effects
@@
 		)
 	)
-	(hierarchical_label "LED2_IN"
+	(hierarchical_label "GND"
+		(shape bidirectional)
+		(at 120.65 69.85 270)
+		(effects
+			(font
+				(size 1.27 1.27)
+			)
+			(justify right)
+		)
+	)
+	(hierarchical_label "LED1_IN"
 		(shape bidirectional)
 		(at 113.03 63.5 180)
@@
 		)
 	)
-	(hierarchical_label "LED2_OUT"
+	(hierarchical_label "LED1_OUT"
 		(shape bidirectional)
 		(at 135.89 63.5 0)
@@
 	(hierarchical_label "GND"
 		(shape bidirectional)
-		(at 120.65 45.72 270)
-		(effects
-			(font
-				(size 1.27 1.27)
-			)
-			(justify right)
-		)
-	)
-	(hierarchical_label "LED4_IN"
-		(shape bidirectional)
-		(at 113.03 110.49 180)
-		(effects
-			(font
-				(size 1.27 1.27)
-			)
-			(justify right)
+		(at 120.65 92.71 270)
+		(effects
+			(font
+				(size 1.27 1.27)
+			)
+			(justify right)
+		)
+	)
+	(hierarchical_label "LED4_OUT"
+		(shape bidirectional)
+		(at 138.43 86.36 0)
+		(effects
+			(font
+				(size 1.27 1.27)
+			)
+			(justify left)
 		)
 	)
 	(hierarchical_label "GND"
 		(shape bidirectional)
-		(at 120.65 69.85 270)
-		(effects
-			(font
-				(size 1.27 1.27)
-			)
-			(justify right)
-		)
-	)
-	(hierarchical_label "LED1_IN"
-		(shape bidirectional)
-		(at 113.03 39.37 180)
-		(effects
-			(font
-				(size 1.27 1.27)
-			)
-			(justify right)
-		)
-	)
-	(hierarchical_label "LED1_OUT"
-		(shape bidirectional)
-		(at 135.89 39.37 0)
-		(effects
-			(font
-				(size 1.27 1.27)
-			)
-			(justify left)
-		)
-	)
-	(hierarchical_label "GND"
-		(shape bidirectional)
-		(at 120.65 92.71 270)
-		(effects
-			(font
-				(size 1.27 1.27)
-			)
-			(justify right)
-		)
-	)
-	(hierarchical_label "LED4_OUT"
-		(shape bidirectional)
-		(at 135.89 110.49 0)
-		(effects
-			(font
-				(size 1.27 1.27)
-			)
-			(justify left)
-		)
-	)
-	(hierarchical_label "GND"
-		(shape bidirectional)
 		(at 120.65 116.84 270)
 		(effects
@@
 	(hierarchical_label "LED3_OUT"
 		(shape bidirectional)
-		(at 135.89 86.36 0)
+		(at 142.24 110.49 0)
 		(effects
 			(font
@@
 	(symbol
 		(lib_id "Device:R")
-		(at 132.08 110.49 90)
+		(at 134.62 86.36 90)
 		(unit 1)
 		(exclude_from_sim no)
@@
 		(fields_autoplaced yes)
 		(property "Reference" "R7"
-			(at 132.08 104.14 90)
+			(at 134.62 80.01 90)
 			(effects
 				(font
@@
 		)
 		(property "Value" "470"
-			(at 132.08 106.68 90)
+			(at 134.62 82.55 90)
 			(effects
 				(font
@@
 		)
 		(property "Footprint" "Resistor_SMD:R_0402_1005Metric_Pad0.72x0.64mm_HandSolder"
-			(at 132.08 112.268 90)
+			(at 134.62 88.138 90)
 			(effects
 				(font
@@
 		)
 		(property "Datasheet" "~"
-			(at 132.08 110.49 0)
+			(at 134.62 86.36 0)
 			(effects
 				(font
@@
 		)
 		(property "Description" "Resistor"
-			(at 132.08 110.49 0)
+			(at 134.62 86.36 0)
 			(effects
 				(font
@@
 	(symbol
 		(lib_id "Device:R")
-		(at 132.08 39.37 90)
+		(at 132.08 63.5 90)
 		(unit 1)
 		(exclude_from_sim no)
@@
 		(fields_autoplaced yes)
 		(property "Reference" "R4"
-			(at 132.08 33.02 90)
+			(at 132.08 57.15 90)
 			(effects
 				(font
@@
 		)
 		(property "Value" "470"
-			(at 132.08 35.56 90)
+			(at 132.08 59.69 90)
 			(effects
 				(font
@@
 		)
 		(property "Footprint" "Resistor_SMD:R_0402_1005Metric_Pad0.72x0.64mm_HandSolder"
-			(at 132.08 41.148 90)
+			(at 132.08 65.278 90)
 			(effects
 				(font
@@
 		)
 		(property "Datasheet" "~"
-			(at 132.08 39.37 0)
+			(at 132.08 63.5 0)
 			(effects
 				(font
@@
 		)
 		(property "Description" "Resistor"
-			(at 132.08 39.37 0)
+			(at 132.08 63.5 0)
 			(effects
 				(font
@@
 	(symbol
 		(lib_id "Device:R")
-		(at 132.08 86.36 90)
+		(at 138.43 110.49 90)
 		(unit 1)
 		(exclude_from_sim no)
@@
 		(fields_autoplaced yes)
 		(property "Reference" "R6"
-			(at 132.08 80.01 90)
+			(at 138.43 104.14 90)
 			(effects
 				(font
@@
 		)
 		(property "Value" "470"
-			(at 132.08 82.55 90)
+			(at 138.43 106.68 90)
 			(effects
 				(font
@@
 		)
 		(property "Footprint" "Resistor_SMD:R_0402_1005Metric_Pad0.72x0.64mm_HandSolder"
-			(at 132.08 88.138 90)
+			(at 138.43 112.268 90)
 			(effects
 				(font
@@
 		)
 		(property "Datasheet" "~"
-			(at 132.08 86.36 0)
+			(at 138.43 110.49 0)
 			(effects
 				(font
@@
 		)
 		(property "Description" "Resistor"
-			(at 132.08 86.36 0)
+			(at 138.43 110.49 0)
 			(effects
 				(font
@@
 	(symbol
 		(lib_id "Device:R")
-		(at 132.08 63.5 90)
+		(at 132.08 39.37 90)
 		(unit 1)
 		(exclude_from_sim no)
@@
 		(fields_autoplaced yes)
 		(property "Reference" "R5"
-			(at 132.08 57.15 90)
+			(at 132.08 33.02 90)
 			(effects
 				(font
@@
 		)
 		(property "Value" "470"
-			(at 132.08 59.69 90)
+			(at 132.08 35.56 90)
 			(effects
 				(font
@@
 		)
 		(property "Footprint" "Resistor_SMD:R_0402_1005Metric_Pad0.72x0.64mm_HandSolder"
-			(at 132.08 65.278 90)
+			(at 132.08 41.148 90)
 			(effects
 				(font
@@
 		)
 		(property "Datasheet" "~"
-			(at 132.08 63.5 0)
+			(at 132.08 39.37 0)
 			(effects
 				(font
@@
 		)
 		(property "Description" "Resistor"
-			(at 132.08 63.5 0)
-			(effects
-				(font
+			(at 132.08 39.37 0)
+			(effects
+				(font
